Commit message: modified file

File: spur_description/robots/spur_robot.urdf.xacro (robot description, xacro)
@@ -2,8 +2,5 @@
 <robot name="spur" xmlns:xacro="http://ros.org/wiki/xacro">
   <xacro:include filename="$(find spur_description)/urdf/base/base.urdf.xacro"/>
-  <!-- ___________________________link joint____________________________ -->
   <link name='base_footprint'/>
-  <xacro:base_macro parent='base_footprint'>
-    <origin xyz='0 0 0'/>
-  </xacro:base_macro>
+  <xacro:base_macro parent='base_footprint'/>
 </robot>

File: spur_description/urdf/base/base.urdf.xacro (robot description, xacro)
@@ -1,4 +1,4 @@
 <?xml version="1.0"?>
-<robot xmlns:xacro="http://ros.org/wiki/xacro">
+<robot name='spur' xmlns:xacro="http://ros.org/wiki/xacro">
   <xacro:include filename="$(find spur_description)/urdf/matelial/materials.urdf.xacro" />
   <xacro:macro name="base_macro" params='parent'>
@@ -72,5 +72,4 @@
 	  <origin xyz='0 0 0'/>
 	</joint>
-<!-- """"""""""""""""""""""""""""""""""""""""""""""""""""""""""""""""""""""""""""""""""""""""" -->
 <!-- """"""""""""""""""""""""""""""""""""""fr""""""""""""""""""""""""""""""""""""""""""""""" -->
         <link name="fr_motor1">
@@ -128,5 +127,4 @@
 	  <origin xyz='0 0 0'/>
 	</joint>
-<!-- """"""""""""""""""""""""""""""""""""""""""""""""""""""""""""""""""""""""""""""""""""""""" -->
 <!-- """"""""""""""""""""""""""""""""""""""bl""""""""""""""""""""""""""""""""""""""""""""""" -->
         <link name="bl_motor1">
@@ -184,5 +182,4 @@
 	  <origin xyz='0 0 0'/>
 	</joint>
-<!-- """"""""""""""""""""""""""""""""""""""""""""""""""""""""""""""""""""""""""""""""""""""""" -->
 <!-- """"""""""""""""""""""""""""""""""""""br""""""""""""""""""""""""""""""""""""""""""""""" -->
         <link name="br_motor1">
@@ -240,5 +237,5 @@
 	  <origin xyz='0 0 0'/>
 	</joint>
-<!-- """"""""""""""""""""""""""""""""""""""""""""""""""""""""""""""""""""""""""""""""""""""""" -->
+<!-- """"""""""""""""""""""""""""""""""""urg"""""""""""""""""""""""""""""""""""""""""""""""""" -->
         <link name='urg_sensor' type='fixed'>
 	  <visual>
